File: CounterModule.brd (EAGLE design)
At the start: 160 x 100.1 mm, 212 parts, among them U1 PCA9547PW, U2 AD5242BRZ100, U3 AD5242BRZ100, U4 AD5242BRZ100, U5 AD5242BRZ100, U6 PTR08060WVD, U7 PTR08060WVD, U8 PTR08060WVD, U9 11AA02E48T-I/TT, X2 0446200002

Commit message: Prototype 2019/03/16 complete reconstruction.
Parts:
- removed R22, R23, R24, R25: (no value), rcl:R0402
- removed R26, R27, R28, R29, R30, R31, R32: 0, rcl:R0402
- removed R33, R37: 0R, rcl:R0402
- removed R38: 10.2K, Panasonic-ERJ2RKF_00:RESC1005X40N
- removed R41: 3.92K, Panasonic-ERJ2RKF_01:RESC1005X40N
- removed S1:P1:Q1, S1:P2:Q1, S1:P3:Q1, S1:P4:Q1, S2:P1:Q1, S2:P2:Q1, S2:P3:Q1, S2:P4:Q1: MUN2211T1, transistor-npn:SC59-BEC
- removed S1:P1:U2, S1:P2:U2, S1:P3:U2, S1:P4:U2, S2:P1:U2, S2:P2:U2, S2:P3:U2, S2:P4:U2: PSSI2021SAY, PSSI2021SAY:SOT353
- added OS1701, OS2701: OSC-OE-CFPS-69, IQD-Frequency-Products:5.0X3.2-4-PAD
- added S1:P1:LED3, S1:P2:LED3, S1:P3:LED3, S1:P4:LED3, S2:P1:LED3, S2:P2:LED3, S2:P3:LED3, S2:P4:LED3: CMD17-21VYC_TR8, CMLighting-CMD17-21VxC_TR8:LED_CMD17-21VYC_TR8
- added S3: 219-02, switch-dil:CTS-219-02
- IC1701, IC2701: value (none) -> MAX14830ETM+
- J1: value (none) -> J1
- R10, R11, R12, R13: value (none) -> 10.2K; device rcl:R0402 -> Panasonic-ERJ2RKF_00:RESC1005X40N
- R14, R15, R16, R17, R18, R19: value 0 -> 10.2K; device rcl:R0402 -> Panasonic-ERJ2RKF_00:RESC1005X40N
- R20, R21: value 0 -> 4.7 kOhm; device rcl:R0402 -> Panasonic-ERJ2RKF_02:RESC1005X40N
- S1:P1:R3, S1:P2:R3, S1:P3:R3, S1:P4:R3, S2:P1:R3, S2:P2:R3, S2:P3:R3, S2:P4:R3: value 221R -> 2K
- S1:P1:U1, S1:P2:U1, S1:P3:U1, S1:P4:U1, S2:P1:U1, S2:P2:U1, S2:P3:U1, S2:P4:U1: value (none) -> CPC1002N
- SV1: value (none) -> SV1
- SV2: value (none) -> SV2
- U9: value 11AA02E48T-I/TT -> 24AA02E48-I/SN; device Microchip-11AA:SOT95P237X112-3N -> Microchip-24AA02E48-I_SN:SOIC127P600X175-8N
- X1: value (none) -> X1
- moved R20 74.6 mm to (47.5, 56.2), flipped to the top, turned to 0 degrees
- moved R21 70.8 mm to (50.0, 56.1), flipped to the top, turned to 180 degrees
- moved R12 38.1 mm to (124.4, 26.0), turned to 90 degrees
- moved R13 38.1 mm to (120.7, 26.1), turned to 90 degrees
- moved R16 35.7 mm to (124.4, 61.6), turned to 90 degrees
- moved R17 35.6 mm to (120.7, 61.6), turned to 90 degrees
- moved C8 27.6 mm to (45.4, 54.0), flipped to the top, turned to 270 degrees
- moved U9 24.0 mm to (48.8, 51.8), flipped to the top, turned to 90 degrees
- moved R19 18.2 mm to (120.8, 79.4), turned to 90 degrees
- moved R15 18.1 mm to (120.8, 43.8), turned to 90 degrees
- moved R18 17.8 mm to (124.4, 79.4), turned to 90 degrees
- moved R14 17.8 mm to (124.5, 43.8), turned to 90 degrees
- moved R11 16.5 mm to (133.2, 17.1), flipped to the top
- moved R10 14.9 mm to (135.7, 18.2), flipped to the top
- moved S2:P1:R3 8.30 mm to (117.5, 54.8), flipped to the top, turned to 180 degrees
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Connections:
- removed net MAC_ID: MICROZED1.JX2_90, R37.1
- removed net N$15: R10.2, R14.1, U2.2
- removed net N$16: R11.2, R16.1, U2.16
- removed net N$17: R22.2, R26.1, U4.2
- removed net N$18: R12.2, R18.1, U3.2
- removed net N$19: R13.2, R20.1, U3.16
- removed net N$20: R23.2, R28.1, U4.16
- removed net N$21: R24.2, R30.1, U5.2
- removed net N$22: R25.2, R32.1, U5.16
- removed net N$6: R37.2, R38.1, U9.1
- removed net S1:P1:GPIO25: S1:P1:Q1.B, S1:P1:U3.11
- removed net S1:P1:LEDFULL: S1:P1:R3.2, S1:P1:U2.2
- removed net S1:P1:SWITCH: S1:P1:Q1.C, S1:P1:U2.3
- removed net S1:P2:GPIO25: S1:P2:Q1.B, S1:P2:U3.11
- removed net S1:P2:LEDFULL: S1:P2:R3.2, S1:P2:U2.2
- removed net S1:P2:SWITCH: S1:P2:Q1.C, S1:P2:U2.3
- removed net S1:P3:GPIO25: S1:P3:Q1.B, S1:P3:U3.11
- removed net S1:P3:LEDFULL: S1:P3:R3.2, S1:P3:U2.2
- removed net S1:P3:SWITCH: S1:P3:Q1.C, S1:P3:U2.3
- removed net S1:P4:GPIO25: S1:P4:Q1.B, S1:P4:U3.11
- removed net S1:P4:LEDFULL: S1:P4:R3.2, S1:P4:U2.2
- removed net S1:P4:SWITCH: S1:P4:Q1.C, S1:P4:U2.3
- removed net S2:P1:GPIO25: S2:P1:Q1.B, S2:P1:U3.11
- removed net S2:P1:LEDFULL: S2:P1:R3.2, S2:P1:U2.2
- removed net S2:P1:SWITCH: S2:P1:Q1.C, S2:P1:U2.3
- removed net S2:P2:GPIO25: S2:P2:Q1.B, S2:P2:U3.11
- removed net S2:P2:LEDFULL: S2:P2:R3.2, S2:P2:U2.2
- removed net S2:P2:SWITCH: S2:P2:Q1.C, S2:P2:U2.3
- removed net S2:P3:GPIO25: S2:P3:Q1.B, S2:P3:U3.11
- removed net S2:P3:LEDFULL: S2:P3:R3.2, S2:P3:U2.2
- removed net S2:P3:SWITCH: S2:P3:Q1.C, S2:P3:U2.3
- removed net S2:P4:GPIO25: S2:P4:Q1.B, S2:P4:U3.11
- removed net S2:P4:LEDFULL: S2:P4:R3.2, S2:P4:U2.2
- removed net S2:P4:SWITCH: S2:P4:Q1.C, S2:P4:U2.3
- removed net VIN_HDR: MICROZED1.JX1_58, MICROZED1.JX1_59
- new net !BRD_ADR0: MICROZED1.JX2_1, R10.2, S3.1
- new net !BRD_ADR1: MICROZED1.JX2_2, R11.2, S3.2
- new net S1:N$6: IC1701.45, OS1701.3
- new net S1:P1:N$6: S1:P1:LED3.1, S1:P1:R3.1
- new net S1:P2:N$6: S1:P2:LED3.1, S1:P2:R3.1
- new net S1:P3:N$6: S1:P3:LED3.1, S1:P3:R3.1
- new net S1:P4:N$6: S1:P4:LED3.1, S1:P4:R3.1
- new net S2:N$6: IC2701.45, OS2701.3
- new net S2:P1:N$6: S2:P1:LED3.1, S2:P1:R3.1
- new net S2:P2:N$6: S2:P2:LED3.1, S2:P2:R3.1
- new net S2:P3:N$6: S2:P3:LED3.1, S2:P3:R3.1
- new net S2:P4:N$6: S2:P4:LED3.1, S2:P4:R3.1
- new net SC5: R20.2, U1.16, U9.6
- new net SD5: R21.1, U1.15, U9.5
- net +3V3: now also OS1701.4, OS2701.4, R10.1, R11.1, R20.1, R21.2, U9.8; no longer R38.2, U9.2
- net +5V: now also MICROZED1.JX1_58, MICROZED1.JX1_59; no longer R14.2, R16.2, R18.2, R20.2, R26.2, R28.2, R30.2, R32.2, R41.2, S1:P1:U2.5, S1:P2:U2.5, S1:P3:U2.5, S1:P4:U2.5, S2:P1:U2.5, S2:P2:U2.5, S2:P3:U2.5, S2:P4:U2.5
- net GND: now also OS1701.2, OS2701.2, S1:P1:LED3.2, S1:P2:LED3.2, S1:P3:LED3.2, S1:P4:LED3.2, S2:P1:LED3.2, S2:P2:LED3.2, S2:P3:LED3.2, S2:P4:LED3.2, S3.3, S3.4, U2.15, U2.3, U3.15, U3.3, U4.15, U4.3, U5.15, U5.3, U9.1, U9.2, U9.4, U9.7; no longer R41.1, S1:P1:Q1.E, S1:P2:Q1.E, S1:P3:Q1.E, S1:P4:Q1.E, S2:P1:Q1.E, S2:P2:Q1.E, S2:P3:Q1.E, S2:P4:Q1.E
- net LED1: now also R12.1; no longer S1:P1:R3.1
- net LED2: now also R13.1; no longer S1:P2:R3.1
- net LED3: now also R14.1; no longer S1:P3:R3.1
- net LED4: now also R15.1; no longer S1:P4:R3.1
- net LED5: now also R16.1; no longer S2:P1:R3.1
- net LED6: now also R17.1; no longer S2:P2:R3.1
- net LED7: now also R18.1; no longer S2:P3:R3.1
- net LED8: now also R19.1; no longer S2:P4:R3.1
- net N$10: now also R18.2; no longer R24.1, R31.1, U5.3
- net N$11: now also R12.2; no longer R10.1, R15.1, U2.3
- net N$12: now also R13.2; no longer R11.1, R17.1, U2.15
- net N$13: now also R15.2; no longer R23.1, R29.1, U4.15
- net N$14: now also R14.2; no longer R22.1, R27.1, U4.3
- net N$4: now also R16.2; no longer R12.1, R19.1, U3.3
- net N$8: now also R17.2; no longer R13.1, R21.1, U3.15
- net N$9: now also R19.2; no longer R25.1, R33.1, U5.15
- net PWR1: now also S1:P1:R3.2
- net PWR2: now also S1:P2:R3.2
- net PWR3: now also S1:P3:R3.2
- net PWR4: now also S1:P4:R3.2
- net PWR5: now also S2:P1:R3.2
- net PWR6: now also S2:P2:R3.2
- net PWR7: now also S2:P3:R3.2
- net PWR8: now also S2:P4:R3.2
- net REXT1: now also S1:P1:U3.11, U2.2; no longer R15.2, S1:P1:U2.4
- net REXT2: now also S1:P2:U3.11, U2.16; no longer R17.2, S1:P2:U2.4
- net REXT3: now also S1:P3:U3.11, U4.2; no longer R27.2, S1:P3:U2.4
- net REXT4: now also S1:P4:U3.11, U4.16; no longer R29.2, S1:P4:U2.4
- net REXT5: now also S2:P1:U3.11, U3.2; no longer R19.2, S2:P1:U2.4
- net REXT6: now also S2:P2:U3.11, U3.16; no longer R21.2, S2:P2:U2.4
- net REXT7: now also S2:P3:U3.11, U5.2; no longer R31.2, S2:P3:U2.4
- net REXT8: now also S2:P4:U3.11, U5.16; no longer R33.2, S2:P4:U2.4
- net VCCIO_EN: no longer U8.1
Routing:
- net +3V3: track 145.0 -> 290.2 mm, vias 44 -> 15
- net VCCIO_EN: track 119.4 -> 0.00 mm, vias 1 -> 0
- net !BRD_ADR0: track 0.00 -> 113.5 mm, vias 0 -> 2
- net !BRD_ADR1: track 0.00 -> 109.4 mm, vias 0 -> 2
- net GND: track 553.4 -> 655.9 mm, vias 76 -> 53
- net S1:P1:GPIO25: track 53.2 -> 0.00 mm, vias 1 -> 0
- net S2:P3:GPIO25: track 50.7 -> 0.00 mm, vias 1 -> 0
- net S1:P3:GPIO25: track 49.0 -> 0.00 mm, vias 1 -> 0
- net +5V: track 148.5 -> 196.2 mm, vias 77 -> 38
- net REXT7: track 1.74 -> 49.2 mm, vias 0 -> 2
- net S2:P1:GPIO25: track 47.1 -> 0.00 mm, vias 2 -> 0
- net REXT1: track 1.73 -> 47.5 mm, vias 0 -> 2
- net REXT5: track 1.74 -> 46.0 mm, vias 0 -> 2
- net REXT3: track 1.74 -> 44.0 mm, vias 0 -> 2
- net S1:P4:GPIO25: track 39.8 -> 0.00 mm, vias 1 -> 0
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Other:
- board text added: "Board Address 1|2|3"
- board text added: "Fast Countermodule Production Sept. 18, 2018 holger.linne@gmx.de"
- board text removed: "Fast Countermodule Prototype 18/08/2017 holger.linne@mpimet.mpg.de (or holger.linne@gmx.de)"
