File: CounterModule.sch (EAGLE design)
At the start: 64 parts, among them U1 PCA9547PW, U2 AD5242BRZ100, U3 AD5242BRZ100, U4 AD5242BRZ100, U5 AD5242BRZ100, U6 PTR08060WVD, U7 PTR08060WVD, U8 PTR08060WVD, U9 11AA02E48T-I/TT, X2 0446200002

Commit message: Prototype 2019/03/16 complete reconstruction.
Parts:
- removed R22, R23, R24, R25: (no value), rcl:R-US_R0402
- removed R26, R27, R28, R29, R30, R31, R32: 0, rcl:R-US_R0402
- removed R33, R37: 0R, rcl:R-US_R0402
- removed R38: 10.2K, Panasonic-ERJ2RKF_00:ERJ-2RKF1022X
- removed R41: 3.92K, Panasonic-ERJ2RKF_01:ERJ-2RKF3921X
- added S3: 219-02, switch-dil:219-02
- J1: value (none) -> J1
- R10, R11, R12, R13: value (none) -> 10.2K; device rcl:R-US_R0402 -> Panasonic-ERJ2RKF_00:ERJ-2RKF1022X
- R14, R15, R16, R17, R18, R19: value 0 -> 10.2K; device rcl:R-US_R0402 -> Panasonic-ERJ2RKF_00:ERJ-2RKF1022X
- R20, R21: value 0 -> 4.7 kOhm; device rcl:R-US_R0402 -> Panasonic-ERJ2RKF_02:ERJ-2RKF4701X
- SV1: value (none) -> SV1
- SV2: value (none) -> SV2
- U9: value 11AA02E48T-I/TT -> 24AA02E48-I/SN; device Microchip-11AA:11AA02E48T-I/TT -> Microchip-24AA02E48-I_SN:24AA02E48-I/SN
- X1: value (none) -> X1
Connections:
- net LED renamed N$6
- removed net GPIO25: U3.B3
- removed net LEDFULL: R3.R2, U2.IOUT
- removed net MAC_ID: MICROZED1-JX2.JX2_LVDS_23_N, R37.1
- removed net N$15: R10.2, R14.1, U2.A1
- removed net N$16: R11.2, R16.1, U2.A2
- removed net N$17: R22.2, R26.1, U4.A1
- removed net N$18: R12.2, R18.1, U3.A1
- removed net N$19: R13.2, R20.1, U3.A2
- removed net N$20: R23.2, R28.1, U4.A2
- removed net N$21: R24.2, R30.1, U5.A1
- removed net N$22: R25.2, R32.1, U5.A2
- removed net N$6 (its old number): R37.2, R38.R1, U9.SOIC
- removed net SWITCH: U2.GND
- new net !BRD_ADR0: MICROZED1-JX2.PMOD_D0, R10.R2, S3.1
- new net !BRD_ADR1: MICROZED1-JX2.PMOD_D1, R11.R2, S3.2
- new net SC5: R20.R2, U1.SC5, U9.SCL
- new net SD5: R21.R1, U1.SD5, U9.SDA
- net +3V3: now also R10.R1, R11.R1, R20.R1, R21.R2; no longer R38.R2
- net +5V: now also MICROZED1-JX1.VIN_HDR@58, MICROZED1-JX1.VIN_HDR@59; no longer R14.2, R16.2, R18.2, R20.2, R26.2, R28.2, R30.2, R32.2, R41.R2, U2.VS
- net GND: now also J1G$2.GND@1, J1G$2.GND@2, J1G$2.GND@3, J1G$2.GND@4, J1G$2.GND@5, J1G$2.GND@6, MICROZED1-JX1.GND@95, S3.3, S3.4, U2.W1, U2.W2, U3.W1, U3.W2, U4.W1, U4.W2, U5.W1, U5.W2, U9.NC, U9.NC1, U9.NC2, U9.NC3; no longer R41.R1
- net LED1: now also R12.R1
- net LED2: now also R13.R1
- net LED3: now also R14.R1
- net LED4: now also R15.R1
- net LED5: now also R16.R1
- net LED6: now also R17.R1
- net LED7: now also R18.R1
- net LED8: now also R19.R1
- net N$10: now also R18.R2; no longer R24.1, R31.1, U5.W1
- net N$11: now also R12.R2; no longer R10.1, R15.1, U2.W1
- net N$12: now also R13.R2; no longer R11.1, R17.1, U2.W2
- net N$13: now also R15.R2; no longer R23.1, R29.1, U4.W2
- net N$14: now also R14.R2; no longer R22.1, R27.1, U4.W1
- net N$4: now also R16.R2; no longer R12.1, R19.1, U3.W1
- net N$8: now also R17.R2; no longer R13.1, R21.1, U3.W2
- net N$9: now also R19.R2; no longer R25.1, R33.1, U5.W2
- net PWR: now also R3.R2
- net REXT: now also U3.B3; no longer U2.REXT
- net REXT1: now also U2.A1; no longer R15.2
- net REXT2: now also U2.A2; no longer R17.2
- net REXT3: now also U4.A1; no longer R27.2
- net REXT4: now also U4.A2; no longer R29.2
- net REXT5: now also U3.A1; no longer R19.2
- net REXT6: now also U3.A2; no longer R21.2
- net REXT7: now also U5.A1; no longer R31.2
- net REXT8: now also U5.A2; no longer R33.2
- net VCCIO_EN: no longer U8.INHIBT
Other:
- note added: "/Users/hll/bypig.bmp"
- note added: "0101100 0x2C"
- note added: "0101101 0x2D"
- note added: "All functionms are connected to the ARM processor using the IIC-bus. Here the processor - bus gets multipülexed to the local busses IIC0 to IIC5 by the multiplexer U1. The modules S1 and S2 contain the serial interface chips."
- note added: "Creative Commons License Attribution 4.0 International (CC BY 4.0) holger.linne@gmx.de"
- note added: "GP0: switch PMT 12V power on/off GP1: switch PMT clock on/off GP2: provide power for tunable LED GP3: switch on/off PCB red LED"
- note added: "System adresses at multiplexer: IIC0: serial chip in S1 (3.3V) IIC1: LED current port 1, 2, 3 and 4 (5V) IIC2: serial chip in S2 (3.3V) IIC3: LED current port 5, 6, 7 and 8 (5V) IIC4: front pannel LED driver (5V) IIC5: MAC address eeprom (3.3V)"
- note added: "System input voltage is 5V, Bank34 (differential input from counter) is set to 2.5V to provide fast LVDS2.5 input to the PL. Bank35 and Bank13 (all other I/O lines) are set to 3.3V."
- note removed: "All functionms are connected to the ARM processor using the IIC-bus. Here the processor - bus gets multipülexed to the local busses IIC0 to IIC4 by the multiplexer U1. The modules S1 and S2 contain the serial interface chips."
- note removed: "Do not populate R10,R11,R12,R13 and R22,R23,R24,R25 !"
- note removed: "System adresses at multiplexer: IIC0: serial chip in S1 (3.3V) IIC1: LED current port 1, 2, 3 and 4 (5V) IIC2: serial chip in S2 (3.3V) IIC3: LED current port 5, 6, 7 and 8 (5V) IIC4: front pannel LED driver (5V)"
- note removed: "System voltage input is 5V, Bank34 (differential input from counter) is set to 2.5V to provide fast LVDS2.5 input to the PL. Bank35 and Bank13 (all other I/O lines) are set to 3.3V."
- moved on the sheet: C8, R40, R8, R9
